Commit message: sherpa = smb clon teleop & spawn funktioniert

File: sherpa_description/urdf/sensor_plugins/smb_imu.gazebo.xacro (robot description, xacro)
@@ -2,5 +2,5 @@
 <!-- This file contains plugins to simulate an Imu sensor attached to the robot. -->
 <!-- Documentation can be found at http://wiki.ros.org/hector_gazebo_plugins -->
-<robot name="sherpa" xmlns:xacro="http://www.ros.org/wiki/xacro">
+<robot name="smb" xmlns:xacro="http://www.ros.org/wiki/xacro">
   <xacro:macro name="IMU" params="base_link simulation">
     <!--                              Imu  Properties 				          	-->
@@ -27,5 +27,5 @@
     <xacro:if value="${simulation}">
     <gazebo>
-      <plugin name="sherpa_imu_plugin" filename="libhector_gazebo_ros_imu.so">
+      <plugin name="smb_imu_plugin" filename="libhector_gazebo_ros_imu.so">
         <updateRate>${imu_update_rate}</updateRate>
         <bodyName>${imu_link}</bodyName>
@@ -65,5 +65,5 @@
         <geometry>
         <!-- <box size="0.04 0.05 0.02"/> -->
-        <mesh filename="package://sherpa_description/urdf/new_payload/meshes/sherpa_imu.dae"/>
+        <mesh filename="package://smb_description/urdf/new_payload/meshes/SMB_imu.dae"/>
       </geometry>
       </visual>
@@ -72,5 +72,5 @@
         <geometry>
           <!-- <box size=".001 .001 .001"/> -->
-          <mesh filename="package://sherpa_description/urdf/new_payload/meshes/sherpa_imu.dae"/>
+          <mesh filename="package://smb_description/urdf/new_payload/meshes/SMB_imu.dae"/>
         </geometry>
       </collision>

File: sherpa_description/urdf/sensor_plugins/smb_velodyne.gazebo.xacro (robot description, xacro)
@@ -1,4 +1,4 @@
 <?xml version="1.0"?>
-<robot name="sherpa" xmlns:xacro="http://www.ros.org/wiki/xacro">
+<robot name="smb" xmlns:xacro="http://www.ros.org/wiki/xacro">
   <xacro:arg name="simulation"   		default="false"/>
   <xacro:arg name="gpu" 		 		default="false"/>

File: sherpa_description/urdf/sherpa.urdf.xacro (robot description, xacro)
@@ -1,29 +1,12 @@
 <?xml version="1.0"?>
-<robot xmlns:xacro="http://www.ros.org/wiki/xacro" name="sherpa">
+<robot xmlns:xacro="http://www.ros.org/wiki/xacro" name="smb">
     <xacro:arg name="lidar" default="true"/>
-    <!-- Fehlende Properties definieren -->
-    <xacro:property name="base_link_name" value="base_link"/>
-    <xacro:property name="wheelRadius" value="0.125"/>
-    <xacro:property name="wheelWidth" value="0.1"/>
-    <xacro:property name="wheelMass" value="1.0"/>
-    <xacro:property name="chassisLength" value="0.6"/>
-    <xacro:property name="chassisWidth" value="0.4"/>
-    <xacro:property name="chassisHeight" value="0.15"/>
-    <xacro:property name="chassisMass" value="10.0"/>
-    <xacro:property name="frontWheelX" value="0.2"/>
-    <xacro:property name="backWheelX" value="-0.2"/>
-    <xacro:property name="wheelClearance" value="0.05"/>
-    <xacro:property name="wheelHeight" value="0.0"/>
-    <xacro:property name="topLength" value="0.5"/>
-    <xacro:property name="topWidth" value="0.35"/>
-    <xacro:property name="topHeight" value="0.1"/>
-    <xacro:property name="topXOffset" value="0.0"/>
-    <xacro:include filename="$(find sherpa_description)/urdf/sherpa_utils.urdf.xacro" />
-    <xacro:include filename="$(find sherpa_description)/urdf/sensor_plugins/sherpa_imu.gazebo.xacro"/>
-    <!--<xacro:include filename="$(find sherpa_description)/urdf/sensor_plugins/sherpa_gps.gazebo.xacro"/> -->
+    <xacro:include filename="$(find smb_description)/urdf/smb_utils.urdf.xacro" />
+    <xacro:include filename="$(find smb_description)/urdf/sensor_plugins/smb_imu.gazebo.xacro"/>
+    <xacro:include filename="$(find smb_description)/urdf/sensor_plugins/smb_gps.gazebo.xacro"/>
     <xacro:if value="$(arg lidar)">
-        <xacro:include filename="$(find sherpa_description)/urdf/sensor_plugins/sherpa_velodyne.gazebo.xacro"/>
+        <xacro:include filename="$(find smb_description)/urdf/sensor_plugins/smb_velodyne.gazebo.xacro"/>
     </xacro:if>
-    <xacro:include filename="$(find sherpa_description)/urdf/sherpa_lidar_mount.urdf.xacro"/>
+    <xacro:include filename="$(find smb_description)/urdf/smb_lidar_mount.urdf.xacro"/>
     <xacro:property name="PI" value="3.1415926535897931"/>
     <!-- Model macros -->
@@ -42,16 +25,12 @@
                 <origin xyz="0 0 0" rpy="0 0 0" />
                 <geometry>
-                    <cylinder length="${wheelWidth}" radius="${wheelRadius}"/>
+                    <cylinder length="${wheelWidth/10}" radius="${wheelRadius}"/>
                 </geometry>
             </collision>
             <visual>
-                <origin xyz="0 0 0" rpy="0 0 0" />
+                <origin xyz="0 0 0" rpy="1.570796 0  0" />
                 <geometry>
-                    <!-- Ersetze Mesh durch primitives Geometrieelement -->
-                    <cylinder length="${wheelWidth}" radius="${wheelRadius}"/>
+                    <mesh filename="package://smb_description/urdf/meshes/wheel.dae" />
                 </geometry>
-                <material name="wheel_material">
-                    <color rgba="0.2 0.2 0.2 1.0"/>
-                </material>
             </visual>
             <inertial>
@@ -98,9 +77,4 @@
                 </material>
             </visual>
-            <inertial>
-                <origin xyz="0 0 0" rpy="0 0 0"/>
-                <mass value="${chassisMass}"/>
-                <xacro:box_inertia m="${chassisMass}" x="${chassisLength}" y="${chassisWidth}" z="${chassisHeight}"/>
-            </inertial>
         </link>
         <link name="top">
@@ -114,16 +88,8 @@
                 <origin xyz="0 0 0" rpy="0 0 0"/>
                 <geometry>
-                    <!-- Ersetze Mesh durch primitives Geometrieelement -->
-                    <box size="${topLength} ${topWidth} ${topHeight}"/>
+                    <!-- <box size="${topLength} ${topWidth} ${topHeight}"/> -->
+                     <mesh filename="package://smb_description/urdf/new_payload/meshes/SMB_step.dae"/>
                 </geometry>
-                <material name="top_material">
-                    <color rgba="0.5 0.5 0.5 1.0"/>
-                </material>
             </visual>
-            <inertial>
-                <origin xyz="0 0 0" rpy="0 0 0"/>
-                <mass value="1.0"/>
-                <xacro:box_inertia m="1.0" x="${topLength}" y="${topWidth}" z="${topHeight}"/>
-            </inertial>
         </link>
         <gazebo reference="top">
@@ -133,28 +99,29 @@
             <material>Gazebo/Red</material>
         </gazebo>
-        <joint name="top_to_base_link" type="fixed">
-            <parent link="${base_link_name}"/>
-            <child link="top"/>
-            <origin xyz="0.0 0.0 ${chassisHeight/2.0}" rpy="0 0 0"/>
-        </joint>
-        <!-- Fixed joint to add dummy inertia link -->
-        <joint name="base_to_base_inertia" type="fixed">
-          <parent link="${base_link_name}"/>
-          <child link="base_inertia"/>
-          <origin xyz="0 0 0" rpy="0 0 0"/>
-        </joint>
-        <!-- Dummy inertia link, because KDL cannot have inertia on the base link -->
-        <link name="base_inertia">
-          <inertial>
-            <origin xyz="0 0 0" rpy="0 0 0"/>
-            <mass value="${chassisMass}"/>
-            <xacro:box_inertia m="${chassisMass}"
-                         x="${chassisLength}"
-                         y="${chassisWidth}"
-                         z="${chassisHeight}"/>
-          </inertial>
-        </link>
+    <joint name="top_to_base_link" type="fixed">
+        <parent link="${base_link_name}"/>
+        <child link="top"/>
+        <!-- <origin xyz="${topXOffset/2.0} 0.0 ${chassisHeight/2.0 + topHeight/2.0}" rpy="0 0 0"/> -->
+        <origin xyz="0.0 0.0 ${chassisHeight/2.0}" rpy="0 0 0"/>
+    </joint>
+    <!-- Fixed joint to add dummy inertia link -->
+    <joint name="base_to_base_inertia" type="fixed">
+      <parent link="${base_link_name}"/>
+      <child link="base_inertia"/>
+      <origin xyz="0 0 0" rpy="0 0 0"/>
+    </joint>
+    <!-- Dummy inertia link, because KDL cannot have inertia on the base link -->
+    <link name="base_inertia">
+      <inertial>
+        <origin xyz="0 0 0" rpy="0 0 0"/>
+        <mass value="${chassisMass}"/>
+        <xacro:box_inertia m="${chassisMass}"
+                     x="${chassisLength}"
+                     y="${chassisWidth}"
+                     z="${chassisHeight}"/>
+      </inertial>
+    </link>
     </xacro:macro>
-    <xacro:macro name="sherpa" params="wheel_joint_type:=continuous lidar:=true simulation:=true">
+    <xacro:macro name="smb" params="wheel_joint_type:=continuous lidar:=true simulation:=true">
         <xacro:chassis/>
         <xacro:wheel prefix="LF" X="${frontWheelX}"
@@ -168,10 +135,11 @@
         <xacro:wheel prefix="LH" X="${backWheelX}"
             Y="${chassisWidth/2+wheelClearance+wheelWidth/2}"
-            wheel_joint_type="${wheel_joint_type}"
-            friction_coeff="0.0" />
+	    wheel_joint_type="${wheel_joint_type}"
+        friction_coeff="0.0" />
         <xacro:wheel prefix="RH" X="${backWheelX}"
             Y="${-chassisWidth/2-wheelClearance-wheelWidth/2}"
             wheel_joint_type="${wheel_joint_type}" />
         <xacro:IMU base_link="${base_link_name}" simulation="${simulation}"/>
+        <!-- <xacro:GPS base_link="base" simulation="${simulation}"/> -->
         <xacro:if value="${lidar}">
             <xacro:LIDAR base_link="${base_link_name}" simulation="${simulation}"/>
@@ -179,5 +147,3 @@
         </xacro:if>
     </xacro:macro>
-    <!-- Instanziieren des Sherpa-Roboters -->
-    <xacro:sherpa wheel_joint_type="continuous" lidar="$(arg lidar)" simulation="true"/>
 </robot>

File: sherpa_description/urdf/sherpa_utils.urdf.xacro (robot description, xacro)
@@ -32,31 +32,31 @@
             />
         </xacro:macro>
-        <!-- Materials -->
-    <material name="black">
-        <color rgba="0.0 0.0 0.0 1.0"/>
-    </material>
-    <material name="dark_grey">
-        <color rgba="0.0 0.0 0.0 0.6"/>
-    </material>
-    <material name="blue">
-        <color rgba="0.0 0.0 0.78 1.0"/>
-    </material>
-    <material name="green">
-        <color rgba="0.0 0.78 0.0 1.0"/>
-    </material>
-    <material name="grey">
-        <color rgba="0.2 0.2 0.2 1.0"/>
-    </material>
-    <material name="orange">
-        <color rgba="1.0 0.42 0.04 1.0"/>
-    </material>
-    <material name="brown">
-        <color rgba="0.87 0.81 0.76 1.0"/>
-    </material>
-    <material name="red">
-        <color rgba="0.78 0.0 0.0 1.0"/>
-    </material>
-    <material name="white">
-        <color rgba="1.0 1.0 1.0 1.0"/>
-    </material>
+    <!-- Materials -->
+        <material name="black">
+            <color rgba="0 0 0 255"/>
+        </material>
+        <material name="dark_grey">
+          <color rgba="0 0 0 155 255"/>
+        </material>
+        <material name="blue">
+            <color rgba="0 0 200 255"/>
+        </material>
+        <material name="green">
+            <color rgba="0 200 0 255"/>
+        </material>
+        <material name="grey">
+            <color rgba="50 50 50 255"/>
+        </material>
+        <material name="orange">
+            <color rgba="255 108 10 255"/>
+        </material>
+        <material name="brown">
+            <color rgba="222 207 195 255"/>
+        </material>
+        <material name="red">
+            <color rgba="200 0 0 255"/>
+        </material>
+        <material name="white">
+            <color rgba="255 255 255 255"/>
+        </material>
   </robot>
