Commit message: further smb to sherpa changes

File: sherpa_description/urdf/sensor_plugins/sherpa_blackfly.gazebo.xacro (robot description, xacro)
@@ -1,4 +1,4 @@
 <?xml version="1.0"?>
-<robot name="smb" xmlns:xacro="http://www.ros.org/wiki/xacro">
+<robot name="sherpa" xmlns:xacro="http://www.ros.org/wiki/xacro">
 <xacro:macro name="blackfly_camera_plugin" params="name rate">
 <gazebo reference="${name}_link">

File: sherpa_description/urdf/sensor_plugins/sherpa_blackfly_stereo.gazebo.xacro (robot description, xacro)
@@ -1,4 +1,4 @@
 <?xml version="1.0"?>
-<robot name="smb" xmlns:xacro="http://www.ros.org/wiki/xacro">
+<robot name="sherpa" xmlns:xacro="http://www.ros.org/wiki/xacro">
 <xacro:macro name="blackfly_camera_stereo_plugin" params="name rate">
 <gazebo reference="${name}_left_link">

File: sherpa_description/urdf/sensor_plugins/sherpa_depth.gazebo.xacro (robot description, xacro)
@@ -1,4 +1,4 @@
 <?xml version="1.0"?>
-<robot name="smb" xmlns:xacro="http://www.ros.org/wiki/xacro">
+<robot name="sherpa" xmlns:xacro="http://www.ros.org/wiki/xacro">
 <xacro:macro name="depth_sensor_plugin" params="name rate">
     <!--                              Imu  Properties 				          	-->
@@ -63,5 +63,5 @@
         <geometry>
         <!-- <box size="0.04 0.05 0.02"/> -->
-        <mesh filename="package://smb_description/urdf/new_payload/meshes/SMB_blackfly.dae"/>
+        <mesh filename="package://sherpa_description/urdf/new_payload/meshes/sherpa_blackfly.dae"/>
       </geometry>
       </visual>
@@ -70,5 +70,5 @@
         <geometry>
           <!-- <box size=".001 .001 .001"/> -->
-          <mesh filename="package://smb_description/urdf/new_payload/meshes/SMB_blackfly.dae"/>
+          <mesh filename="package://sherpa_description/urdf/new_payload/meshes/sherpa_blackfly.dae"/>
         </geometry>
       </collision>

File: sherpa_description/urdf/sensor_plugins/sherpa_gps.gazebo.xacro (robot description, xacro)
@@ -2,5 +2,5 @@
 <!-- This file contains a plugin to simulate a gps sensor attached to the robot. -->
 <!-- Documentation can be found at http://wiki.ros.org/hector_gazebo_plugins -->
-<robot name="smb" xmlns:xacro="http://www.ros.org/wiki/xacro">
+<robot name="sherpa" xmlns:xacro="http://www.ros.org/wiki/xacro">
 <xacro:macro name="GPS" params="base_link simulation:=false">
    <!--                              Gps  Properties 	           				-->
@@ -28,5 +28,5 @@
     <xacro:if value="${simulation}">
     <gazebo>
-      <plugin name="smb_gps_plugin" filename="libhector_gazebo_ros_gps.so">
+      <plugin name="sherpa_gps_plugin" filename="libhector_gazebo_ros_gps.so">
         <updateRate>${gps_update_rate}</updateRate>
         <bodyName>${gps_link}</bodyName>

File: sherpa_description/urdf/sensor_plugins/sherpa_imu.gazebo.xacro (robot description, xacro)
@@ -2,5 +2,5 @@
 <!-- This file contains plugins to simulate an Imu sensor attached to the robot. -->
 <!-- Documentation can be found at http://wiki.ros.org/hector_gazebo_plugins -->
-<robot name="smb" xmlns:xacro="http://www.ros.org/wiki/xacro">
+<robot name="sherpa" xmlns:xacro="http://www.ros.org/wiki/xacro">
   <xacro:macro name="IMU" params="base_link simulation">
     <!--                              Imu  Properties 				          	-->
@@ -27,5 +27,5 @@
     <xacro:if value="${simulation}">
     <gazebo>
-      <plugin name="smb_imu_plugin" filename="libhector_gazebo_ros_imu.so">
+      <plugin name="sherpa_imu_plugin" filename="libhector_gazebo_ros_imu.so">
         <updateRate>${imu_update_rate}</updateRate>
         <bodyName>${imu_link}</bodyName>
@@ -65,5 +65,5 @@
         <geometry>
         <!-- <box size="0.04 0.05 0.02"/> -->
-        <mesh filename="package://smb_description/urdf/new_payload/meshes/SMB_imu.dae"/>
+        <mesh filename="package://sherpa_description/urdf/new_payload/meshes/sherpa_imu.dae"/>
       </geometry>
       </visual>
@@ -72,5 +72,5 @@
         <geometry>
           <!-- <box size=".001 .001 .001"/> -->
-          <mesh filename="package://smb_description/urdf/new_payload/meshes/SMB_imu.dae"/>
+          <mesh filename="package://sherpa_description/urdf/new_payload/meshes/sherpa_imu.dae"/>
         </geometry>
       </collision>

File: sherpa_description/urdf/sensor_plugins/sherpa_mono.gazebo.xacro (robot description, xacro)
@@ -2,5 +2,5 @@
 <!-- This file contains plugins to simulate an Imu sensor attached to the robot. -->
 <!-- Documentation can be found at http://wiki.ros.org/hector_gazebo_plugins -->
-<robot name="smb" xmlns:xacro="http://www.ros.org/wiki/xacro">
+<robot name="sherpa" xmlns:xacro="http://www.ros.org/wiki/xacro">
   <xacro:macro name="mono_cam" params="base_link simulation">
     <!--                              Imu  Properties 				          	-->

File: sherpa_description/urdf/sensor_plugins/sherpa_odometry.gazebo.xacro (robot description, xacro)
@@ -1,8 +1,8 @@
 <?xml version="1.0"?>
-<robot xmlns:xacro="http://www.ros.org/wiki/xacro" name="smb">
+<robot xmlns:xacro="http://www.ros.org/wiki/xacro" name="sherpa">
 <xacro:macro name="odometry_plugin" params="sensor_link topic_name odom_frame:=camera_odom_frame child_odom_frame:=camera_pose_frame publish_tf:=true rate:=20 max_linear_speed_before_settle:=0.001 max_angular_speed_before_settle:=0.001">
     <gazebo>
-        <plugin name="smb_odometry_plugin" filename="libodometry_source_plugin.so">
-            <robotNamespace>smb</robotNamespace>
+        <plugin name="sherpa_odometry_plugin" filename="libodometry_source_plugin.so">
+            <robotNamespace>sherpa</robotNamespace>
             <bodyName>${sensor_link}</bodyName>
             <topicName>${topic_name}</topicName>

File: sherpa_description/urdf/sensor_plugins/sherpa_velodyne.gazebo.xacro (robot description, xacro)
@@ -1,4 +1,4 @@
 <?xml version="1.0"?>
-<robot name="smb" xmlns:xacro="http://www.ros.org/wiki/xacro">
+<robot name="sherpa" xmlns:xacro="http://www.ros.org/wiki/xacro">
   <xacro:arg name="simulation"   		default="false"/>
   <xacro:arg name="gpu" 		 		default="false"/>

File: sherpa_description/urdf/sherpa.urdf.xacro (robot description, xacro)
@@ -1,12 +1,12 @@
 <?xml version="1.0"?>
-<robot xmlns:xacro="http://www.ros.org/wiki/xacro" name="smb">
+<robot xmlns:xacro="http://www.ros.org/wiki/xacro" name="sherpa">
     <xacro:arg name="lidar" default="true"/>
-    <xacro:include filename="$(find smb_description)/urdf/smb_utils.urdf.xacro" />
-    <xacro:include filename="$(find smb_description)/urdf/sensor_plugins/smb_imu.gazebo.xacro"/>
-    <xacro:include filename="$(find smb_description)/urdf/sensor_plugins/smb_gps.gazebo.xacro"/>
+    <xacro:include filename="$(find sherpa_description)/urdf/sherpa_utils.urdf.xacro" />
+    <xacro:include filename="$(find sherpa_description)/urdf/sensor_plugins/sherpa_imu.gazebo.xacro"/>
+    <xacro:include filename="$(find sherpa_description)/urdf/sensor_plugins/sherpa_gps.gazebo.xacro"/>
     <xacro:if value="$(arg lidar)">
-        <xacro:include filename="$(find smb_description)/urdf/sensor_plugins/smb_velodyne.gazebo.xacro"/>
+        <xacro:include filename="$(find sherpa_description)/urdf/sensor_plugins/sherpa_velodyne.gazebo.xacro"/>
     </xacro:if>
-    <xacro:include filename="$(find smb_description)/urdf/smb_lidar_mount.urdf.xacro"/>
+    <xacro:include filename="$(find sherpa_description)/urdf/sherpa_lidar_mount.urdf.xacro"/>
     <xacro:property name="PI" value="3.1415926535897931"/>
     <!-- Model macros -->
@@ -31,5 +31,5 @@
                 <origin xyz="0 0 0" rpy="1.570796 0  0" />
                 <geometry>
-                    <mesh filename="package://smb_description/urdf/meshes/wheel.dae" />
+                    <mesh filename="package://sherpa_description/urdf/meshes/wheel.dae" />
                 </geometry>
             </visual>
@@ -89,5 +89,5 @@
                 <geometry>
                     <!-- <box size="${topLength} ${topWidth} ${topHeight}"/> -->
-                     <mesh filename="package://smb_description/urdf/new_payload/meshes/SMB_step.dae"/>
+                     <mesh filename="package://sherpa_description/urdf/new_payload/meshes/sherpa_step.dae"/>
                 </geometry>
             </visual>
@@ -123,5 +123,5 @@
     </link>
     </xacro:macro>
-    <xacro:macro name="smb" params="wheel_joint_type:=continuous lidar:=true simulation:=true">
+    <xacro:macro name="sherpa" params="wheel_joint_type:=continuous lidar:=true simulation:=true">
         <xacro:chassis/>
         <xacro:wheel prefix="LF" X="${frontWheelX}"

File: sherpa_description/urdf/sherpa_big_properties.urdf.xacro (robot description, xacro)
@@ -1,4 +1,4 @@
 <?xml version="1.0"?>
-<robot xmlns:xacro="http://www.ros.org/wiki/xacro" name="smb">
+<robot xmlns:xacro="http://www.ros.org/wiki/xacro" name="sherpa">
     <xacro:property name="base_link_name" value="base_link"/>
     <xacro:property name="chassisHeight" value="0.197"/>

File: sherpa_description/urdf/sherpa_lidar_mount.urdf.xacro (robot description, xacro)
@@ -2,5 +2,5 @@
 <!-- This file contains plugins to simulate an Imu sensor attached to the robot. -->
 <!-- Documentation can be found at http://wiki.ros.org/hector_gazebo_plugins -->
-<robot name="smb" xmlns:xacro="http://www.ros.org/wiki/xacro">
+<robot name="sherpa" xmlns:xacro="http://www.ros.org/wiki/xacro">
   <xacro:macro name="lidar_mount" params="base_link">
     <!--                              Imu  Properties 				          	-->
@@ -11,5 +11,5 @@
       <visual>
         <geometry>
-          <mesh filename="package://smb_description/urdf/new_payload/meshes/SMB_lidar_mount.dae"/>
+          <mesh filename="package://sherpa_description/urdf/new_payload/meshes/sherpa_lidar_mount.dae"/>
         </geometry>
       </visual>

File: sherpa_description/urdf/sherpa_ros_control.gazebo.xacro (robot description, xacro)
@@ -1,6 +1,6 @@
 <?xml version="1.0"?>
 <!-- This file contains the Gazebo controller interface. -->
-<robot name="smb" xmlns:xacro="http://www.ros.org/wiki/xacro">
-  <xacro:macro name="smb_ros_control_plugin" params="description_name
+<robot name="sherpa" xmlns:xacro="http://www.ros.org/wiki/xacro">
+  <xacro:macro name="sherpa_ros_control_plugin" params="description_name
                                                         broadcast_tf
                                                         robot_namespace">

File: sherpa_description/urdf/sherpa_ros_skid_steer.gazebo.xacro (robot description, xacro)
@@ -1,6 +1,6 @@
 <?xml version="1.0"?>
 <!-- This file contains the Gazebo controller interface. -->
-<robot name="smb" xmlns:xacro="http://www.ros.org/wiki/xacro">
-  <xacro:macro name="smb_ros_skid_steer_plugin" params="description_name
+<robot name="sherpa" xmlns:xacro="http://www.ros.org/wiki/xacro">
+  <xacro:macro name="sherpa_ros_skid_steer_plugin" params="description_name
                                                         broadcast_tf
                                                         robot_namespace">

File: sherpa_description/urdf/sherpa_standalone.urdf.xacro (robot description, xacro)
@@ -1,4 +1,4 @@
 <?xml version="1.0"?>
-<robot xmlns:xacro="http://www.ros.org/wiki/xacro" name="smb">
+<robot xmlns:xacro="http://www.ros.org/wiki/xacro" name="sherpa">
   <!-- Arguments -->
   <xacro:arg name="wheel_joint_type"          default="fixed"/> <!-- continuous for gazebo -->
@@ -10,10 +10,10 @@
   <xacro:property name="lidar" value="$(arg lidar)"/>
       <!-- Includes -->
-  <xacro:include filename="$(find smb_description)/urdf/smb_big_properties.urdf.xacro" />
-  <xacro:include filename="$(find smb_description)/urdf/smb.urdf.xacro"/>
-  <xacro:smb wheel_joint_type="$(arg wheel_joint_type)" simulation="$(arg simulation)"/>
+  <xacro:include filename="$(find sherpa_description)/urdf/sherpa_big_properties.urdf.xacro" />
+  <xacro:include filename="$(find sherpa_description)/urdf/sherpa.urdf.xacro"/>
+  <xacro:sherpa wheel_joint_type="$(arg wheel_joint_type)" simulation="$(arg simulation)"/>
   <!-- Handle gazebo plugins -->
-  <xacro:include filename="$(find smb_description)/urdf/smb_ros_skid_steer.gazebo.xacro"/>
-  <xacro:smb_ros_skid_steer_plugin description_name="$(arg description_name_xacro)"
+  <xacro:include filename="$(find sherpa_description)/urdf/sherpa_ros_skid_steer.gazebo.xacro"/>
+  <xacro:sherpa_ros_skid_steer_plugin description_name="$(arg description_name_xacro)"
       broadcast_tf="$(arg publish_tf)" robot_namespace="$(arg robot_namespace)"/>
   <gazebo>
