Commit message: delete old Lidar and implement rp lidar for simulation

File: sherpa_description/urdf/sensor_plugins/sherpa_rplidar.gazebo.xacro (robot description, xacro)
@@ -2,9 +2,9 @@
 <robot xmlns:xacro="http://www.ros.org/wiki/xacro">
   <xacro:macro name="RPLIDAR" params="base_link:=base_link simulation:=true">
-    <!-- RPLidar Link -->
+    <!-- RPLidar Link - Position erhöht von 0.2 auf 0.3 Meter für besseren Überblick -->
     <joint name="rplidar_joint" type="fixed">
       <parent link="${base_link}"/>
       <child link="rplidar_link"/>
-      <origin xyz="0.0 0.0 0.2" rpy="0 0 0"/>
+      <origin xyz="0.0 0.0 0.3" rpy="0 0 0"/>
     </joint>
     <link name="rplidar_link">
@@ -32,4 +32,6 @@
       <gazebo reference="rplidar_link">
         <material>Gazebo/Black</material>
+        <!-- Self-collision deaktivieren -->
+        <selfCollide>false</selfCollide>
         <sensor type="ray" name="rslidar">
           <pose>0 0 0 0 0 0</pose>
@@ -46,5 +48,6 @@
             </scan>
             <range>
-              <min>0.15</min>
+              <!-- Minimalen Scanbereich erhöht von 0.15 auf 0.35 Meter -->
+              <min>0.35</min>
               <max>12.0</max>
               <resolution>0.01</resolution>
@@ -59,5 +62,6 @@
             <topicName>scan</topicName>
             <frameName>rplidar_link</frameName>
-            <min_range>0.15</min_range>
+            <!-- Auch hier den minimalen Scanbereich anpassen -->
+            <min_range>0.35</min_range>
             <max_range>12.0</max_range>
             <gaussianNoise>0.008</gaussianNoise>

File: sherpa_description/urdf/sherpa.urdf.xacro (robot description, xacro)
@@ -5,8 +5,4 @@
     <xacro:include filename="$(find sherpa_description)/urdf/sensor_plugins/sherpa_imu.gazebo.xacro"/>
     <xacro:include filename="$(find sherpa_description)/urdf/sensor_plugins/sherpa_rplidar.gazebo.xacro"/>
-    <xacro:if value="$(arg lidar)">
-        <xacro:include filename="$(find sherpa_description)/urdf/sensor_plugins/sherpa_velodyne.gazebo.xacro"/>
-    </xacro:if>
-    <xacro:include filename="$(find sherpa_description)/urdf/sherpa_lidar_mount.urdf.xacro"/>
     <xacro:property name="PI" value="3.1415926535897931"/>
     <!-- Model macros -->
@@ -142,8 +138,4 @@
         <xacro:IMU base_link="${base_link_name}" simulation="${simulation}"/>
         <xacro:RPLIDAR base_link="${base_link_name}" simulation="${simulation}"/>
-        <xacro:if value="${lidar}">
-            <xacro:LIDAR base_link="${base_link_name}" simulation="${simulation}"/>
-            <xacro:lidar_mount base_link="${base_link_name}"/>
-        </xacro:if>
     </xacro:macro>
 </robot>
