Commit message: basic wheel geometries

File: sherpa_description/urdf/sherpa.urdf.xacro (robot description, xacro)
@@ -29,7 +29,7 @@
             </collision>
             <visual>
-                <origin xyz="0 0 0" rpy="1.570796 0  0" />
+                <origin xyz="0 0 0" rpy="0 0 0" />
                 <geometry>
-                    <mesh filename="package://sherpa_description/urdf/meshes/wheel.dae" />
+                    <cylinder length="${wheelWidth/10}" radius="${wheelRadius}"/>
                 </geometry>
             </visual>

Commit message: basic mecanum implementation

File: sherpa_description/urdf/sherpa.urdf.xacro (robot description, xacro)
@@ -7,4 +7,58 @@
     <xacro:property name="PI" value="3.1415926535897931"/>
     <!-- Model macros -->
+    <xacro:macro name="mecanum_wheel" params="prefix X Y wheel_joint_type friction_coeff:=0.2 transmission_reduction:=1 roller_angle:=0" >
+        <joint name="${prefix}_WHEEL_JOINT" type="${wheel_joint_type}">
+            <parent link="${base_link_name}"/>
+            <child link="${prefix}_WHEEL"/>
+            <origin xyz="${X} ${Y} ${wheelHeight - chassisHeight/2.0}" rpy="-${0.5*PI} 0 0" />
+            <axis xyz="0 0 1" rpy="0 0 0" />
+            <dynamics damping="1.0" friction="0.0"/>
+            <limit effort="1" velocity="1"/>
+            <joint_properties damping="0.2" friction="0.2"/>
+        </joint>
+        <link name="${prefix}_WHEEL">
+            <collision>
+                <origin xyz="0 0 0" rpy="0 0 0" />
+                <geometry>
+                    <cylinder length="${wheelWidth/10}" radius="${wheelRadius}"/>
+                </geometry>
+            </collision>
+            <visual>
+                <origin xyz="0 0 0" rpy="0 0 ${roller_angle}" />
+                <geometry>
+                    <!-- Using a mesh for better visualization of mecanum wheel -->
+                    <mesh filename="package://sherpa_description/meshes/mecanum_wheel.dae" scale="${wheelRadius*5} ${wheelRadius*5} ${wheelRadius*5}"/>
+                </geometry>
+                <material name="dark_grey"/>
+            </visual>
+            <inertial>
+                <origin xyz="0 0 0" rpy="0 0 0" />
+                <mass value="${wheelMass}"/>
+                <xacro:cylinder_inertia m="${wheelMass}" r="${wheelRadius}" h="${wheelWidth}"/>
+            </inertial>
+        </link>
+        <gazebo reference="${prefix}_WHEEL">
+            <!-- Special settings for mecanum wheels -->
+            <mu1 value="${friction_coeff}"/>
+            <mu2 value="${friction_coeff}"/>
+            <!-- Using the roller angle to set the friction direction -->
+            <fdir1 value="0 ${sin(roller_angle)} ${cos(roller_angle)}"/>
+            <kp>10000000.0</kp>
+            <kd>1.0</kd>
+            <minDepth>0.005</minDepth>
+            <maxVel>100.0</maxVel>
+            <material>Gazebo/DarkGrey</material>
+        </gazebo>
+        <transmission name="${prefix}_WHEEL_TRANS" type="SimpleTransmission">
+            <type>transmission_interface/SimpleTransmission</type>
+            <joint name="${prefix}_WHEEL_JOINT">
+                <hardwareInterface>hardware_interface/VelocityJointInterface</hardwareInterface>
+            </joint>
+            <actuator name="${prefix}_ACTUATOR">
+                <mechanicalReduction>${transmission_reduction}</mechanicalReduction>
+            </actuator>
+        </transmission>
+    </xacro:macro>
+    <!-- Keeping the original wheel macro for backward compatibility -->
     <xacro:macro name="wheel" params="prefix X Y wheel_joint_type friction_coeff:=0.2 transmission_reduction:=1" >
         <joint name="${prefix}_WHEEL_JOINT" type="${wheel_joint_type}">
@@ -121,19 +175,28 @@
     <xacro:macro name="sherpa" params="wheel_joint_type:=continuous lidar:=true simulation:=true">
         <xacro:chassis/>
-        <xacro:wheel prefix="LF" X="${frontWheelX}"
+        <!-- Front left wheel - 45 degree roller angle -->
+        <xacro:mecanum_wheel prefix="LF" X="${frontWheelX}"
             Y="${chassisWidth/2+wheelClearance+wheelWidth/2}"
             wheel_joint_type="${wheel_joint_type}"
-            friction_coeff="0.5" />
-        <xacro:wheel prefix="RF" X="${frontWheelX}"
+            friction_coeff="0.5"
+            roller_angle="-0.785" /> <!-- -45 degrees in radians -->
+        <!-- Front right wheel - -45 degree roller angle -->
+        <xacro:mecanum_wheel prefix="RF" X="${frontWheelX}"
             Y="${-chassisWidth/2-wheelClearance-wheelWidth/2}"
             wheel_joint_type="${wheel_joint_type}"
-            friction_coeff="0.5"/>
-        <xacro:wheel prefix="LH" X="${backWheelX}"
+            friction_coeff="0.5"
+            roller_angle="0.785" /> <!-- 45 degrees in radians -->
+        <!-- Rear left wheel - 45 degree roller angle, but opposite to front right -->
+        <xacro:mecanum_wheel prefix="LH" X="${backWheelX}"
             Y="${chassisWidth/2+wheelClearance+wheelWidth/2}"
-	    wheel_joint_type="${wheel_joint_type}"
-        friction_coeff="0.0" />
-        <xacro:wheel prefix="RH" X="${backWheelX}"
+            wheel_joint_type="${wheel_joint_type}"
+            friction_coeff="0.5"
+            roller_angle="0.785" /> <!-- 45 degrees in radians -->
+        <!-- Rear right wheel - -45 degree roller angle, but opposite to front left -->
+        <xacro:mecanum_wheel prefix="RH" X="${backWheelX}"
             Y="${-chassisWidth/2-wheelClearance-wheelWidth/2}"
-            wheel_joint_type="${wheel_joint_type}" />
+            wheel_joint_type="${wheel_joint_type}"
+            friction_coeff="0.5"
+            roller_angle="-0.785" /> <!-- -45 degrees in radians -->
         <xacro:IMU base_link="${base_link_name}" simulation="${simulation}"/>
         <xacro:RPLIDAR base_link="${base_link_name}" simulation="${simulation}"/>

File: sherpa_description/urdf/sherpa_ros_mecanum.gazebo.xacro (robot description, xacro)
@@ -1,12 +1,11 @@
 <?xml version="1.0"?>
-<!-- This file contains the Gazebo controller interface. -->
+<!-- This file contains the Gazebo controller interface for mecanum wheels. -->
 <robot name="sherpa" xmlns:xacro="http://www.ros.org/wiki/xacro">
-  <xacro:macro name="sherpa_ros_skid_steer_plugin" params="description_name
+  <xacro:macro name="sherpa_mecanum_drive_plugin" params="description_name
                                                         broadcast_tf
                                                         robot_namespace">
   <xacro:arg name="base_cmd_topic_name" default="cmd_vel"/>
     <gazebo>
-      <!-- Changed from skid_steer_drive to mecanum_drive -->
-      <plugin name="gazebo_ros_control" filename="libgazebo_ros_planar_move.so">
+      <plugin name="mecanum_controller" filename="libgazebo_ros_planar_move.so">
         <robotNamespace>${robot_namespace}</robotNamespace>
         <commandTopic>$(arg base_cmd_topic_name)</commandTopic>
@@ -15,5 +14,4 @@
         <odometryRate>20.0</odometryRate>
         <robotBaseFrame>${base_link_name}</robotBaseFrame>
-        <broadcastTF>${broadcast_tf}</broadcastTF>
         <publishOdomTF>${broadcast_tf}</publishOdomTF>
         <publishWheelTF>false</publishWheelTF>
@@ -24,4 +22,12 @@
       </plugin>
     </gazebo>
+    <!-- Add joint state controller -->
+    <gazebo>
+      <plugin name="joint_state_publisher" filename="libgazebo_ros_joint_state_publisher.so">
+        <jointName>LF_WHEEL_JOINT, RF_WHEEL_JOINT, LH_WHEEL_JOINT, RH_WHEEL_JOINT</jointName>
+        <updateRate>50.0</updateRate>
+        <robotNamespace>${robot_namespace}</robotNamespace>
+      </plugin>
+    </gazebo>
   </xacro:macro>
 </robot>

File: sherpa_description/urdf/sherpa_standalone.urdf.xacro (robot description, xacro)
@@ -2,5 +2,5 @@
 <robot xmlns:xacro="http://www.ros.org/wiki/xacro" name="sherpa">
   <!-- Arguments -->
-  <xacro:arg name="wheel_joint_type"          default="fixed"/> <!-- continuous for gazebo -->
+  <xacro:arg name="wheel_joint_type"          default="continuous"/> <!-- Changed from 'fixed' to 'continuous' for mecanum wheels -->
   <xacro:arg name="simulation"                default="false"/>
   <xacro:arg name="lidar"                     default="true"/>
@@ -13,7 +13,7 @@
   <xacro:include filename="$(find sherpa_description)/urdf/sherpa.urdf.xacro"/>
   <xacro:sherpa wheel_joint_type="$(arg wheel_joint_type)" simulation="$(arg simulation)"/>
-  <!-- Handle gazebo plugins -->
-  <xacro:include filename="$(find sherpa_description)/urdf/sherpa_ros_skid_steer.gazebo.xacro"/>
-  <xacro:sherpa_ros_skid_steer_plugin description_name="$(arg description_name_xacro)"
+  <!-- Handle gazebo plugins - Changed from skid steer to mecanum drive -->
+  <xacro:include filename="$(find sherpa_description)/urdf/sherpa_ros_mecanum.gazebo.xacro"/>
+  <xacro:sherpa_mecanum_drive_plugin description_name="$(arg description_name_xacro)"
       broadcast_tf="$(arg publish_tf)" robot_namespace="$(arg robot_namespace)"/>
   <gazebo>

Commit message: import meshes wrong orientation

File: sherpa_description/urdf/sherpa.urdf.xacro (robot description, xacro)
@@ -17,4 +17,14 @@
             <joint_properties damping="0.2" friction="0.2"/>
         </joint>
+        <xacro:property name="wheel_mesh" value="package://sherpa_description/meshes/front_left_wheel_1.stl"/>
+        <xacro:if value="${prefix == 'RF'}">
+            <xacro:property name="wheel_mesh" value="package://sherpa_description/meshes/front_right_wheel_1.stl"/>
+        </xacro:if>
+        <xacro:if value="${prefix == 'LH'}">
+            <xacro:property name="wheel_mesh" value="package://sherpa_description/meshes/rear_left_wheel_1.stl"/>
+        </xacro:if>
+        <xacro:if value="${prefix == 'RH'}">
+            <xacro:property name="wheel_mesh" value="package://sherpa_description/meshes/rear_right_wheel_1.stl"/>
+        </xacro:if>
         <link name="${prefix}_WHEEL">
             <collision>
@@ -25,8 +35,7 @@
             </collision>
             <visual>
-                <origin xyz="0 0 0" rpy="0 0 ${roller_angle}" />
-                <geometry>
-                    <!-- Using a mesh for better visualization of mecanum wheel -->
-                    <mesh filename="package://sherpa_description/meshes/mecanum_wheel.dae" scale="${wheelRadius*5} ${wheelRadius*5} ${wheelRadius*5}"/>
+                <origin xyz="0 0 0" rpy="-${0.5*PI} 0 ${roller_angle}" />
+                <geometry>
+                    <mesh filename="${wheel_mesh}" scale="0.001 0.001 0.001"/>
                 </geometry>
                 <material name="dark_grey"/>
@@ -122,4 +131,13 @@
                 <geometry>
                     <box size="${chassisLength} ${chassisWidth} ${chassisHeight}"/>
+                </geometry>
+                <material name="base_material">
+                    <color rgba="0.8 0.0 0.1 1.0"/>
+                </material>
+            </visual>
+            <visual>
+                <origin xyz="0 0 0" rpy="0 0 0"/>
+                <geometry>
+                    <mesh filename="package://sherpa_description/meshes/base_link.stl" scale="0.001 0.001 0.001"/>
                 </geometry>
                 <material name="base_material">

Commit message: visual wheel rotation

File: sherpa_description/urdf/sherpa.urdf.xacro (robot description, xacro)
@@ -35,5 +35,5 @@
             </collision>
             <visual>
-                <origin xyz="0 0 0" rpy="-${0.5*PI} 0 ${roller_angle}" />
+                <origin xyz="0 0 0" rpy="0 -${0.5*PI} 0" />
                 <geometry>
                     <mesh filename="${wheel_mesh}" scale="0.001 0.001 0.001"/>
